File: pcb/io-module/mcu.kicad_sch (KiCad schematic)
At the start: 28 parts, among them J1 SWD Header, SW1 SKRPABE010, U1 STM32C051G8Ux, Y1 ECS-480-10-37B2-RWN-TR

Commit message: Updated parts and IO power connection
Parts:
- removed D1, D2, D3, D4: Blue, CRGM Passive:LED_0603_1608Metric, symbol Device:LED_Small
- removed JP3, JP4: (no value), CRGM Connector:SolderJumper-2_P1.3mm_Open_RoundedPad1.0x1.5mm, symbol Jumper:SolderJumper_2_Open
- added D1, D2, D3, D4: Blue, CRGM Passive:LED_0603_1608Metric, symbol CRGM Passive:LED_Small
- added JP3, JP4: SolderJumper_2_Open, CRGM Connector:SolderJumper-2_P1.3mm_Open_RoundedPad1.0x1.5mm, symbol CRGM Connector:SolderJumper_2_Open
- JP1, JP2: value (none) -> SolderJumper_2_Open
Connections:
- net A0: now also JP3.2 (B)
- net A1: now also JP4.2 (B)
- net GND: now also JP3.1 (A), JP4.1 (A)
- net LED1: now also D1.1 (K)
- net LED2: now also D2.1 (K)
- net LED3: now also D3.1 (K)
- net LED4: now also D4.1 (K)
- net at R4.2: now also D2.2 (A)
- net at R3.2: now also D1.2 (A)
- net at R6.2: now also D4.2 (A)
- net at R5.2: now also D3.2 (A)
Other:
- moved on the sheet: JP1, JP2, R1, R2
