File: pcb/io-module/power.kicad_sch (KiCad schematic)
At the start: 17 parts

Commit message: Updated parts and IO power connection
Parts:
- removed D12, D13, D14: Blue, CRGM Passive:LED_0603_1608Metric, symbol Device:LED_Small
- added D12, D13, D14: Blue, CRGM Passive:LED_0603_1608Metric, symbol CRGM Passive:LED_Small
- D10: MN TECH PUBLIC -> Nexperia; MPN TPSP3022-01ETG -> PESD5V5C1BLYL
- D11: MN FUXINSEMI -> (none); MPN LESD8D3.3CAT5G -> (none)
- JP6, JP7, JP8: value (none) -> SolderJumper_2_Bridged; symbol Jumper:SolderJumper_2_Bridged -> CRGM Connector:SolderJumper_2_Bridged
Connections:
- net V3.3LED: now also D13.2 (A)
- net V5LED: now also D12.2 (A)
- net VIOLED: now also D14.2 (A)
- net at JP7.2 (B): now also D13.1 (K)
- net at JP8.2 (B): now also D14.1 (K)
- net at JP6.2 (B): now also D12.1 (K)
