File: pcb/io-module.kicad_pcb (KiCad board)
At the start: 4 copper layers, 50 x 25 mm, 127 parts, among them J1 SWD Header, J12 Conn_02x02_Odd_Even, SW1 SKRPABE010, U1 STM32C051G8Ux, Y1 ECS-480-10-37B2-RWN-TR

Commit message: change version tag
Other:
- board text added: "<<>>"
- board text removed: "vX.Y"
Changed lines of the file:
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@@
 		)
 	)
-	(gr_text "vX.Y"
+	(gr_text "<<>>"
 		(at 91.45 97.8 0)
 		(layer "F.SilkS")
@@
 			)
 		)
-		(render_cache "vX.Y" 0
-			(polygon
-				(pts
-					(xy 89.981857 98.215) (xy 89.700367 97.471891) (xy 90.004266 97.471891) (xy 90.140065 97.932472)
-					(xy 90.146904 97.932472) (xy 90.282703 97.471891) (xy 90.561445 97.471891) (xy 90.277146 98.215)
-				)
-			)
-			(polygon
-				(pts
-					(xy 91.65089 98.215) (xy 91.270909 98.215) (xy 91.0931 97.915375) (xy 91.089742 97.915375) (xy 90.911933 98.215)
-					(xy 90.559979 98.215) (xy 90.905644 97.703433) (xy 90.593502 97.24792) (xy 90.972139 97.24792)
-					(xy 91.117708 97.4943) (xy 91.121127 97.4943) (xy 91.2681 97.24792) (xy 91.618772 97.24792) (xy 91.305225 97.704837)
-				)
-			)
-			(polygon
-				(pts
-					(xy 91.729842 98.215) (xy 91.729842 97.932472) (xy 92.030504 97.932472) (xy 92.030504 98.215)
-				)
-			)
-			(polygon
-				(pts
-					(xy 92.815745 98.215) (xy 92.502443 98.215) (xy 92.502443 97.839781) (xy 92.118554 97.24792) (xy 92.478873 97.24792)
-					(xy 92.663704 97.568489) (xy 92.667062 97.568489) (xy 92.851893 97.24792) (xy 93.193955 97.24792)
-					(xy 92.815745 97.839781)
+		(render_cache "<<>>" 0
+			(polygon
+				(pts
+					(xy 89.937343 97.849063) (xy 90.436209 98.031085) (xy 90.436209 98.234112) (xy 89.697314 97.949813)
+					(xy 89.697314 97.746908) (xy 90.436209 97.461205) (xy 90.436209 97.665575)
+				)
+			)
+			(polygon
+				(pts
+					(xy 90.860581 97.849063) (xy 91.359447 98.031085) (xy 91.359447 98.234112) (xy 90.620552 97.949813)
+					(xy 90.620552 97.746908) (xy 91.359447 97.461205) (xy 91.359447 97.665575)
+				)
+			)
+			(polygon
+				(pts
+					(xy 92.28409 97.949813) (xy 91.545194 98.234112) (xy 91.545194 98.031085) (xy 92.04406 97.849063)
+					(xy 91.545194 97.665575) (xy 91.545194 97.461205) (xy 92.28409 97.746908)
+				)
+			)
+			(polygon
+				(pts
+					(xy 93.207328 97.949813) (xy 92.468432 98.234112) (xy 92.468432 98.031085) (xy 92.967298 97.849063)
+					(xy 92.468432 97.665575) (xy 92.468432 97.461205) (xy 93.207328 97.746908)
 				)
 			)
@@
 		)
 	)
-	(gr_text "vX.Y"
+	(gr_text "<<>>"
 		(at 89.7 97.325 0)
 		(layer "B.SilkS")
@@
 			(justify mirror)
 		)
-		(render_cache "vX.Y" 0
-			(polygon
-				(pts
-					(xy 91.168142 97.74) (xy 91.449632 96.996891) (xy 91.145733 96.996891) (xy 91.009934 97.457472)
-					(xy 91.003095 97.457472) (xy 90.867296 96.996891) (xy 90.588554 96.996891) (xy 90.872853 97.74)
-				)
-			)
-			(polygon
-				(pts
-					(xy 89.499109 97.74) (xy 89.87909 97.74) (xy 90.056899 97.440375) (xy 90.060257 97.440375) (xy 90.238066 97.74)
-					(xy 90.59002 97.74) (xy 90.244355 97.228433) (xy 90.556497 96.77292) (xy 90.17786 96.77292) (xy 90.032291 97.0193)
-					(xy 90.028872 97.0193) (xy 89.881899 96.77292) (xy 89.531227 96.77292) (xy 89.844774 97.229837)
-				)
-			)
-			(polygon
-				(pts
-					(xy 89.420157 97.74) (xy 89.420157 97.457472) (xy 89.119495 97.457472) (xy 89.119495 97.74)
-				)
-			)
-			(polygon
-				(pts
-					(xy 88.334254 97.74) (xy 88.647556 97.74) (xy 88.647556 97.364781) (xy 89.031445 96.77292) (xy 88.671126 96.77292)
-					(xy 88.486295 97.093489) (xy 88.482937 97.093489) (xy 88.298106 96.77292) (xy 87.956044 96.77292)
-					(xy 88.334254 97.364781)
-				)
-			)
+		(render_cache "<<>>" 0
+			(polygon
+				(pts
+					(xy 91.212656 97.374063) (xy 90.71379 97.556085) (xy 90.71379 97.759112) (xy 91.452685 97.474813)
+					(xy 91.452685 97.271908) (xy 90.71379 96.986205) (xy 90.71379 97.190575)
+				)
+			)
+			(polygon
+				(pts
+					(xy 90.289418 97.374063) (xy 89.790552 97.556085) (xy 89.790552 97.759112) (xy 90.529447 97.474813)
+					(xy 90.529447 97.271908) (xy 89.790552 96.986205) (xy 89.790552 97.190575)
+				)
+			)
+			(polygon
+				(pts
+					(xy 88.865909 97.474813) (xy 89.604805 97.759112) (xy 89.604805 97.556085) (xy 89.105939 97.374063)
+					(xy 89.604805 97.190575) (xy 89.604805 96.986205) (xy 88.865909 97.271908)
+				)
+			)
+			(polygon
+				(pts
+					(xy 87.942671 97.474813) (xy 88.681567 97.759112) (xy 88.681567 97.556085) (xy 88.182701 97.374063)
+					(xy 88.681567 97.190575) (xy 88.681567 96.986205) (xy 87.942671 97.271908)
+				)
+			)
