File: pcb/io-module.kicad_pcb (KiCad board)
At the start: 4 copper layers, 50 x 25 mm, 127 parts, among them J1 SWD Header, J12 Conn_02x02_Odd_Even, SW1 SKRPABE010, U1 STM32C051G8Ux, Y1 ECS-480-10-37B2-RWN-TR

Commit message: Updated renders
Changed <<tag>> to vX.Y
Other:
- board text removed: "<<>>"
Changed lines of the file:
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@@
 		)
 	)
-	(gr_text "<<>>"
+	(gr_text "vX.Y"
 		(at 89.7 97.325 0)
 		(layer "B.SilkS")
@@
 			(justify mirror)
 		)
-		(render_cache "<<>>" 0
+		(render_cache "vX.Y" 0
 			(polygon
 				(pts
-					(xy 91.212656 97.374063) (xy 90.71379 97.556085) (xy 90.71379 97.759112) (xy 91.452685 97.474813)
-					(xy 91.452685 97.271908) (xy 90.71379 96.986205) (xy 90.71379 97.190575)
+					(xy 91.168142 97.74) (xy 91.449632 96.996891) (xy 91.145733 96.996891) (xy 91.009934 97.457472)
+					(xy 91.003095 97.457472) (xy 90.867296 96.996891) (xy 90.588554 96.996891) (xy 90.872853 97.74)
 				)
 			)
 			(polygon
 				(pts
-					(xy 90.289418 97.374063) (xy 89.790552 97.556085) (xy 89.790552 97.759112) (xy 90.529447 97.474813)
-					(xy 90.529447 97.271908) (xy 89.790552 96.986205) (xy 89.790552 97.190575)
+					(xy 89.499109 97.74) (xy 89.87909 97.74) (xy 90.056899 97.440375) (xy 90.060257 97.440375) (xy 90.238066 97.74)
+					(xy 90.59002 97.74) (xy 90.244355 97.228433) (xy 90.556497 96.77292) (xy 90.17786 96.77292) (xy 90.032291 97.0193)
+					(xy 90.028872 97.0193) (xy 89.881899 96.77292) (xy 89.531227 96.77292) (xy 89.844774 97.229837)
 				)
 			)
 			(polygon
 				(pts
-					(xy 88.865909 97.474813) (xy 89.604805 97.759112) (xy 89.604805 97.556085) (xy 89.105939 97.374063)
-					(xy 89.604805 97.190575) (xy 89.604805 96.986205) (xy 88.865909 97.271908)
+					(xy 89.420157 97.74) (xy 89.420157 97.457472) (xy 89.119495 97.457472) (xy 89.119495 97.74)
 				)
 			)
 			(polygon
 				(pts
-					(xy 87.942671 97.474813) (xy 88.681567 97.759112) (xy 88.681567 97.556085) (xy 88.182701 97.374063)
-					(xy 88.681567 97.190575) (xy 88.681567 96.986205) (xy 87.942671 97.271908)
+					(xy 88.334254 97.74) (xy 88.647556 97.74) (xy 88.647556 97.364781) (xy 89.031445 96.77292) (xy 88.671126 96.77292)
+					(xy 88.486295 97.093489) (xy 88.482937 97.093489) (xy 88.298106 96.77292) (xy 87.956044 96.77292)
+					(xy 88.334254 97.364781)
 				)
 			)
