File: pcb/interface.kicad_sch (KiCad schematic)
At the start: 33 parts

Commit message: Fixed directories
Parts:
- removed JP5: (no value), CRGM Connector:SolderJumper-2_P2.0mm_Bridged_RoundedPad1.0x1.5mm, symbol Jumper:SolderJumper_2_Bridged
- removed JP9: (no value), CRGM Connector:SolderJumper-2_P1.3mm_Open_RoundedPad1.0x1.5mm, symbol CRGM Connector:SolderJumper_2_Open
- added J12: Conn_02x02_Odd_Even, CRGM Connector:PinHeader_2x02_P1.27mm_Vertical_SMD, symbol Connector_Generic:Conn_02x02_Odd_Even
- D5: MN TECH PUBLIC -> Nexperia; MPN TPSP3022-01ETG -> PESD5V5C1BLYL
- D6, D7, D8, D9: MN FUXINSEMI -> (none); MPN LESD8D3.3CAT5G -> (none)
Connections:
- net +3.3V: now also J12.1 (Pin_1)
- net +5V: now also J12.3 (Pin_3)
- net SERVO1 renamed IO1
- net SERVO2 renamed IO2
- net SERVO3 renamed IO3
- net SERVO4 renamed IO4
- net VSERVO renamed VIO
- net VIO: now also J12.2 (Pin_2), J12.4 (Pin_4)
Other:
- note added: "I/O"
- note removed: "Optional"
- note removed: "Servo"
- company: (none) -> CRG Makes
- title: Servo Module -> I/O Module
- moved on the sheet: D5, J6

Commit message: Updated connector PN, MPN, and model
Parts:
- J12: Digikey (none) -> 609-3692-2-ND; LCSC (none) -> C5160758; LCSC1 (none) -> C3975185; MN (none) -> DEALON; MPN (none) -> DZ127S-22-04-55; Mouser (none) -> 649-202112100004C4LF
Changed lines of the file:
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@@
 			)
 		)
-		(property "Datasheet" ""
+		(property "Datasheet" "https://cdn.amphenol-cs.com/media/wysiwyg/files/documentation/datasheet/boardwiretoboard/bwb_minitek127_btb.pdf"
 			(at 82.55 132.08 0)
 			(hide yes)
@@
 			)
 		)
-		(property "MN" ""
+		(property "MN" "DEALON"
 			(at 82.55 132.08 0)
 			(hide yes)
@@
 			)
 		)
-		(property "MPN" ""
+		(property "MPN" "DZ127S-22-04-55"
 			(at 82.55 132.08 0)
 			(hide yes)
@@
 			)
 		)
-		(property "Digikey" ""
+		(property "Digikey" "609-3692-2-ND"
 			(at 82.55 132.08 0)
 			(hide yes)
@@
 			)
 		)
-		(property "Mouser" ""
+		(property "Mouser" "649-202112100004C4LF"
 			(at 82.55 132.08 0)
 			(hide yes)
@@
 			)
 		)
-		(property "LCSC" ""
+		(property "LCSC" "C5160758"
 			(at 82.55 132.08 0)
 			(hide yes)
+			(show_name no)
+			(do_not_autoplace no)
+			(effects
+				(font
+					(size 1.27 1.27)
+				)
+			)
+		)
+		(property "LCSC1" "C3975185"
+			(at 82.55 132.08 0)
+			(hide yes)

Commit message: fixes #1 and fixes #2
Parts:
- removed TP15, TP16: (no value), CRGM Mechanical:TestPoint_Pad_D1.0mm, symbol Connector:TestPoint
Other:
- moved on the sheet: J7, J8
