File: pcb/mcu.kicad_sch (KiCad schematic)
At the start: 28 parts, among them J1 SWD Header, SW1 SKRPABE010, U1 STM32C051G8Ux, Y1 ECS-480-10-37B2-RWN-TR

Commit message: Fixed directories
Parts:
- removed D1, D2, D3, D4: Blue, CRGM Passive:LED_0603_1608Metric, symbol Device:LED_Small
- removed JP3, JP4: (no value), CRGM Connector:SolderJumper-2_P1.3mm_Open_RoundedPad1.0x1.5mm, symbol Jumper:SolderJumper_2_Open
- added D1, D2, D3, D4: Blue, CRGM Passive:LED_0603_1608Metric, symbol CRGM Passive:LED_Small
- added JP3, JP4: SolderJumper_2_Open, CRGM Connector:SolderJumper-2_P1.3mm_Open_RoundedPad1.0x1.5mm, symbol CRGM Connector:SolderJumper_2_Open
- JP1, JP2: value (none) -> SolderJumper_2_Open
Connections:
- net A0: now also JP3.2 (B)
- net A1: now also JP4.2 (B)
- net GND: now also JP3.1 (A), JP4.1 (A)
- net LED1: now also D1.1 (K)
- net LED2: now also D2.1 (K)
- net LED3: now also D3.1 (K)
- net LED4: now also D4.1 (K)
- net at R4.2: now also D2.2 (A)
- net at R3.2: now also D1.2 (A)
- net at R6.2: now also D4.2 (A)
- net at R5.2: now also D3.2 (A)
- net SERVO1 renamed IO1
- net SERVO2 renamed IO2
- net SERVO3 renamed IO3
- net SERVO4 renamed IO4
Other:
- company: (none) -> CRG Makes
- title: Servo Module -> I/O Module
- moved on the sheet: JP1, JP2, R1, R2

Commit message: admin changes after prod 1.0
Parts:
- D1, D2, D3, D4: MPN (none) -> XL-1608UBC-04
Changed lines of the file:
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@@
+			)
+		)
+		(property "MPN" "XL-1608UBC-04"
+			(at 166.37 50.8 90)
+			(hide yes)
+			(show_name no)
+			(do_not_autoplace no)
+			(effects
+				(font
+					(size 1.27 1.27)
+				)
 			)
 		)
@@
 			)
 		)
+		(property "MPN" "XL-1608UBC-04"
+			(at 160.02 50.8 90)
+			(hide yes)
+			(show_name no)
+			(do_not_autoplace no)
+			(effects
+				(font
+					(size 1.27 1.27)
+				)
+			)
+		)
 		(pin "1"
 		)
@@
 		(property "Sim.Pins" "1=K 2=A"
 			(at 163.83 50.8 0)
+			(hide yes)
+			(show_name no)
+			(do_not_autoplace no)
+			(effects
+				(font
+					(size 1.27 1.27)
+				)
+			)
+		)
+		(property "MPN" "XL-1608UBC-04"
+			(at 153.67 50.8 90)
 			(hide yes)
 			(show_name no)
@@
 			(hide yes)
 			(show_name no)
+			(do_not_autoplace no)
+			(effects
+				(font
+					(size 1.27 1.27)
+				)
+			)
+		)
+		(property "MPN" "XL-1608UBC-04"
+			(at 172.72 50.8 90)
+			(hide yes)
+			(show_name no)

Commit message: fixes #1 and fixes #2
Parts:
- added D15: Blue, CRGM Passive:LED_0603_1608Metric, symbol CRGM Passive:LED_Small
- added R10: 1K, CRGM Passive:R_0603_1608Metric, symbol Device:R_Small
Connections:
- net +3.3V: now also R10.1
- net STATUS: now reaches U1.22 (PA15)
- net STATUS: now also D15.1 (K)
- new net: D15.2 (A), R10.2
- no-connect marks 9 -> 8
Other:
- moved on the sheet: JP1, JP2, JP3, JP4, R1, R2
