File: pcb/power.kicad_sch (KiCad schematic)
At the start: 17 parts

Commit message: Fixed directories
Parts:
- removed D12, D13, D14: Blue, CRGM Passive:LED_0603_1608Metric, symbol Device:LED_Small
- added D12, D13, D14: Blue, CRGM Passive:LED_0603_1608Metric, symbol CRGM Passive:LED_Small
- D10: MN TECH PUBLIC -> Nexperia; MPN TPSP3022-01ETG -> PESD5V5C1BLYL
- D11: MN FUXINSEMI -> (none); MPN LESD8D3.3CAT5G -> (none)
- JP6, JP7, JP8: value (none) -> SolderJumper_2_Bridged; symbol Jumper:SolderJumper_2_Bridged -> CRGM Connector:SolderJumper_2_Bridged
Connections:
- net V3.3LED: now also D13.2 (A)
- net V5LED: now also D12.2 (A)
- net at JP7.2 (B): now also D13.1 (K)
- net at JP8.2 (B): now also D14.1 (K)
- net at JP6.2 (B): now also D12.1 (K)
- net VSERVO renamed VIO
- net VSERVOLED renamed VIOLED
- net VIOLED: now also D14.2 (A)
Other:
- title: Servo Module -> I/O Module

Commit message: admin changes after prod 1.0
Parts:
- D12, D13, D14: Digikey (none) -> 5962-XL-1608UBC-04TR-ND; LCSC (none) -> C965807; MN (none) -> XINGLIGHT; MPN (none) -> XL-1608UBC-04
Changed lines of the file:
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@@
 			)
 		)
-		(property "Datasheet" ""
+		(property "Datasheet" "https://optoelectronics.liteon.com/upload/download/DS-22-99-0224/LTST-C190TBKT.PDF"
 			(at 114.3 45.72 0)
 			(hide yes)
@@
 		(property "Sim.Pins" "1=K 2=A"
 			(at 124.46 45.72 0)
+			(hide yes)
+			(show_name no)
+			(do_not_autoplace no)
+			(effects
+				(font
+					(size 1.27 1.27)
+				)
+			)
+		)
+		(property "Digikey" "5962-XL-1608UBC-04TR-ND"
+			(at 114.3 45.72 90)
+			(hide yes)
+			(show_name no)
+			(do_not_autoplace no)
+			(effects
+				(font
+					(size 1.27 1.27)
+				)
+			)
+		)
+		(property "LCSC" "C965807"
+			(at 114.3 45.72 90)
+			(hide yes)
+			(show_name no)
+			(do_not_autoplace no)
+			(effects
+				(font
+					(size 1.27 1.27)
+				)
+			)
+		)
+		(property "MN" "XINGLIGHT"
+			(at 114.3 45.72 90)
+			(hide yes)
+			(show_name no)
+			(do_not_autoplace no)
+			(effects
+				(font
+					(size 1.27 1.27)
+				)
+			)
+		)
+		(property "MPN" "XL-1608UBC-04"
+			(at 114.3 45.72 90)
 			(hide yes)
 			(show_name no)
@@
 			)
 		)
-		(property "Datasheet" ""
+		(property "Datasheet" "https://optoelectronics.liteon.com/upload/download/DS-22-99-0224/LTST-C190TBKT.PDF"
 			(at 135.89 45.72 0)
 			(hide yes)
@@
 		(property "Sim.Pins" "1=K 2=A"
 			(at 146.05 45.72 0)
+			(hide yes)
+			(show_name no)
+			(do_not_autoplace no)
+			(effects
+				(font
+					(size 1.27 1.27)
+				)
+			)
+		)
+		(property "Digikey" "5962-XL-1608UBC-04TR-ND"
+			(at 135.89 45.72 90)
+			(hide yes)
+			(show_name no)
+			(do_not_autoplace no)
+			(effects
+				(font
+					(size 1.27 1.27)
+				)
+			)
+		)
+		(property "LCSC" "C965807"
+			(at 135.89 45.72 90)
+			(hide yes)
+			(show_name no)
+			(do_not_autoplace no)
+			(effects
+				(font
+					(size 1.27 1.27)
+				)
+			)
+		)
+		(property "MN" "XINGLIGHT"
+			(at 135.89 45.72 90)
+			(hide yes)
+			(show_name no)
+			(do_not_autoplace no)
+			(effects
+				(font
+					(size 1.27 1.27)
+				)
+			)
+		)
+		(property "MPN" "XL-1608UBC-04"
+			(at 135.89 45.72 90)
 			(hide yes)
 			(show_name no)
@@
 			)
 		)
-		(property "Datasheet" ""
+		(property "Datasheet" "https://optoelectronics.liteon.com/upload/download/DS-22-99-0224/LTST-C190TBKT.PDF"
 			(at 125.73 45.72 0)
 			(hide yes)
@@
 			(hide yes)
 			(show_name no)
+			(do_not_autoplace no)
+			(effects
+				(font
+					(size 1.27 1.27)
+				)
+			)
+		)
+		(property "Digikey" "5962-XL-1608UBC-04TR-ND"
+			(at 125.73 45.72 90)
+			(hide yes)
+			(show_name no)
+			(do_not_autoplace no)
+			(effects
+				(font
+					(size 1.27 1.27)
+				)
+			)
+		)
+		(property "LCSC" "C965807"
+			(at 125.73 45.72 90)
+			(hide yes)
+			(show_name no)
+			(do_not_autoplace no)
+			(effects
+				(font
+					(size 1.27 1.27)
+				)
+			)
+		)
+		(property "MN" "XINGLIGHT"
+			(at 125.73 45.72 90)
+			(hide yes)
+			(show_name no)
+			(do_not_autoplace no)
+			(effects
+				(font
+					(size 1.27 1.27)
+				)
+			)
+		)
+		(property "MPN" "XL-1608UBC-04"
+			(at 125.73 45.72 90)
+			(hide yes)
+			(show_name no)

Commit message: fixes #1 and fixes #2
Connections:
- net +3.3V: now also J10.1 (V3), J9.1 (V3); no longer J10.4 (V3), J9.4 (V3)
- net +5V: now also J10.4 (V5), J9.4 (V5); no longer J10.1 (V5), J9.1 (V5)
Changed lines of the file:
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@@
-			)
-		)
-		(property "WVDC" ""
-			(at 77.47 39.37 0)
-			(hide yes)
-			(show_name no)
-			(do_not_autoplace no)
-			(effects
-				(font
-					(size 1.27 1.27)
-				)
 			)
 		)
@@
 			(hide yes)
 			(show_name no)
-			(do_not_autoplace no)
-			(effects
-				(font
-					(size 1.27 1.27)
-				)
-			)
-		)
-		(property "WVDC" ""
-			(at 48.26 39.37 0)
-			(hide yes)
-			(show_name no)
