File: pcb/requirements.kicad_sch (KiCad schematic)
At the start: 10 parts

Commit message: Fixed directories
Parts:
- LOGO1: now in the parts list
- LOGO2: footprint CRGM Logos:Aquarius Logo 3.5mm -> CRGM Logos:Aquarius Logo 5mm; now in the parts list
Other:
- company: (none) -> CRG Makes
- title: Servo Module -> I/O Module
Changed lines of the file:
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@@
 	(paper "A4")
 	(title_block
-		(title "Servo Module")
+		(title "I/O Module")
 		(date "<<release-date>>")
 		(rev "<<tag>>")
+		(company "CRG Makes")
 		(comment 1 "<<hash>>")
 	)
@@
 		)
 	)
-	(text_box "BASIC\n\n* STM32C0 Processor\n* 48MHz Crystal\n* Adafruit Seesaw Protocol\n* Four Servo Ports\n* Power In/Out Ports\n* Optional Pull Ups for I2C\n* I2C Address Selection (2-bits)\n"
+	(text_box "BASIC\n\n* STM32C0 Processor\n* 48MHz Crystal\n* Adafruit Seesaw Protocol\n* Four I/O Ports\n* Power In/Out Ports\n* Optional Pull Ups for I2C\n* I2C Address Selection (2-bits)\n"
 		(exclude_from_sim yes)
 		(at 19.05 32.385 0)
@@
 		)
 	)
-	(text_box "Interfaces:\n* 2 - QWICC\n* 2 - Aquarius Power\n* 1 - Servo Power Input\n* 1 - Serial\n* 1 - Prg/Debug Port\n\nOUTPUT:\n* 4 - Servo Out\n\n"
+	(text_box "Interfaces:\n* 2 - QWICC\n* 2 - Aquarius Power\n* 1 - Servo Power Input\n* 1 - Serial\n* 1 - Prg/Debug Port\n\nOUTPUT:\n* 4 - I/O Out\n\n"
 		(exclude_from_sim yes)
 		(at 161.29 32.385 0)
@@
 		)
 	)
-	(text_box "Servo Specifications\n\n* 5V, 90g\n* 0-180 Degrees\n* Standard PWM\n* Servo Power Connector\n* Servo Power Indicator\n* Servo Status Indicators\n* Bulk and Decoupling Caps"
+	(text_box "I/O Specifications\n\n* 5V or I/O Power\n* Power Connector\n* Power Indicator\n* Status Indicators\n* Bulk and Decoupling Caps"
 		(exclude_from_sim yes)
 		(at 90.17 32.385 0)
@@
 		)
 		(instances
-			(project "servo-module"
+			(project "io-module"
 				(path "/445c1fff-2e1a-48b1-a91f-a137832edebf/5454c337-e679-4d27-a394-0abf4144d85b"
 					(reference "H1")
@@
 		(body_style 1)
 		(exclude_from_sim no)
-		(in_bom no)
+		(in_bom yes)
 		(on_board yes)
 		(in_pos_files yes)
@@
 			)
 		)
-		(property "Footprint" "CRGM Logos:Aquarius Logo 3.5mm"
+		(property "Footprint" "CRGM Logos:Aquarius Logo 5mm"
 			(at 38.354 189.738 0)
 			(hide yes)
@@
 			)
 		)
-		(property "MPN" ""
-			(at 36.83 186.69 0)
-			(show_name no)
-			(do_not_autoplace no)
-			(effects
-				(font
-					(size 1.27 1.27)
-				)
-			)
-		)
-		(property "LCSC" ""
-			(at 36.83 186.69 0)
-			(hide yes)
-			(show_name no)
-			(do_not_autoplace no)
-			(effects
-				(font
-					(size 1.27 1.27)
-				)
-			)
-		)
-		(property "Digikey" ""
-			(at 36.83 186.69 0)
-			(hide yes)
-			(show_name no)
-			(do_not_autoplace no)
-			(effects
-				(font
-					(size 1.27 1.27)
-				)
-			)
-		)
-		(property "Mouser" ""
-			(at 36.83 186.69 0)
-			(hide yes)
-			(show_name no)
-			(do_not_autoplace no)
-			(effects
-				(font
-					(size 1.27 1.27)
-				)
-			)
-		)
-		(property "WVDC" ""
-			(at 36.83 186.69 0)
-			(hide yes)
-			(show_name no)
-			(do_not_autoplace no)
-			(effects
-				(font
-					(size 1.27 1.27)
-				)
-			)
-		)
 		(instances
-			(project "servo-module"
+			(project "io-module"
 				(path "/445c1fff-2e1a-48b1-a91f-a137832edebf/5454c337-e679-4d27-a394-0abf4144d85b"
 					(reference "LOGO2")
@@
 		)
 		(instances
-			(project "servo-module"
+			(project "io-module"
 				(path "/445c1fff-2e1a-48b1-a91f-a137832edebf/5454c337-e679-4d27-a394-0abf4144d85b"
 					(reference "H3")
@@
 		)
 		(instances
-			(project "servo-module"
+			(project "io-module"
 				(path "/445c1fff-2e1a-48b1-a91f-a137832edebf/5454c337-e679-4d27-a394-0abf4144d85b"
 					(reference "LOGO4")
@@
 		)
 		(instances
-			(project "servo-module"
+			(project "io-module"
 				(path "/445c1fff-2e1a-48b1-a91f-a137832edebf/5454c337-e679-4d27-a394-0abf4144d85b"
 					(reference "#PWR01")
@@
 		)
 		(instances
-			(project "servo-module"
+			(project "io-module"
 				(path "/445c1fff-2e1a-48b1-a91f-a137832edebf/5454c337-e679-4d27-a394-0abf4144d85b"
 					(reference "LOGO6")
@@
 		)
 		(instances
-			(project "servo-module"
+			(project "io-module"
 				(path "/445c1fff-2e1a-48b1-a91f-a137832edebf/5454c337-e679-4d27-a394-0abf4144d85b"
 					(reference "H2")
@@
 		)
 		(instances
-			(project "servo-module"
+			(project "io-module"
 				(path "/445c1fff-2e1a-48b1-a91f-a137832edebf/5454c337-e679-4d27-a394-0abf4144d85b"
 					(reference "LOGO3")
@@
 		(body_style 1)
 		(exclude_from_sim no)
-		(in_bom no)
+		(in_bom yes)
 		(on_board yes)
 		(in_pos_files yes)
@@
 			)
 		)
-		(property "MPN" ""
-			(at 25.4 186.69 0)
-			(show_name no)
-			(do_not_autoplace no)
-			(effects
-				(font
-					(size 1.27 1.27)
-				)
-			)
-		)
-		(property "LCSC" ""
-			(at 25.4 186.69 0)
-			(hide yes)
-			(show_name no)
-			(do_not_autoplace no)
-			(effects
-				(font
-					(size 1.27 1.27)
-				)
-			)
-		)
-		(property "Digikey" ""
-			(at 25.4 186.69 0)
-			(hide yes)
-			(show_name no)
-			(do_not_autoplace no)
-			(effects
-				(font
-					(size 1.27 1.27)
-				)
-			)
-		)
-		(property "Mouser" ""
-			(at 25.4 186.69 0)
-			(hide yes)
-			(show_name no)
-			(do_not_autoplace no)
-			(effects
-				(font
-					(size 1.27 1.27)
-				)
-			)
-		)
-		(property "WVDC" ""
-			(at 25.4 186.69 0)
-			(hide yes)
-			(show_name no)
-			(do_not_autoplace no)
-			(effects
-				(font
-					(size 1.27 1.27)
-				)
-			)
-		)
 		(instances
-			(project "servo-module"
+			(project "io-module"
 				(path "/445c1fff-2e1a-48b1-a91f-a137832edebf/5454c337-e679-4d27-a394-0abf4144d85b"
 					(reference "LOGO1")
@@
 		)
 		(instances
-			(project "servo-module"
+			(project "io-module"
 				(path "/445c1fff-2e1a-48b1-a91f-a137832edebf/5454c337-e679-4d27-a394-0abf4144d85b"
 					(reference "LOGO5")
@@
 		)
 		(instances
-			(project "servo-module"
+			(project "io-module"
 				(path "/445c1fff-2e1a-48b1-a91f-a137832edebf/5454c337-e679-4d27-a394-0abf4144d85b"
 					(reference "H4")

Commit message: fixes #1 and fixes #2
Parts:
- LOGO5: footprint CRGM Logos:Roxy 4mm -> CRGM Logos:Roxy 3.5mm
Changed lines of the file:
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@@
+			)
+		)
+		(property "MN" ""
+			(at 36.83 186.69 0)
+			(hide yes)
+			(show_name no)
+			(do_not_autoplace no)
+			(effects
+				(font
+					(size 1.27 1.27)
+				)
+			)
+		)
+		(property "MPN" ""
+			(at 36.83 186.69 0)
+			(hide yes)
+			(show_name no)
+			(do_not_autoplace no)
+			(effects
+				(font
+					(size 1.27 1.27)
+				)
+			)
+		)
+		(property "Digikey" ""
+			(at 36.83 186.69 0)
+			(hide yes)
+			(show_name no)
+			(do_not_autoplace no)
+			(effects
+				(font
+					(size 1.27 1.27)
+				)
+			)
+		)
+		(property "Mouser" ""
+			(at 36.83 186.69 0)
+			(hide yes)
+			(show_name no)
+			(do_not_autoplace no)
+			(effects
+				(font
+					(size 1.27 1.27)
+				)
+			)
+		)
+		(property "LCSC" ""
+			(at 36.83 186.69 0)
+			(hide yes)
+			(show_name no)
+			(do_not_autoplace no)
+			(effects
+				(font
+					(size 1.27 1.27)
+				)
 			)
 		)
@@
 			)
 		)
+		(property "MN" ""
+			(at 85.09 186.69 0)
+			(hide yes)
+			(show_name no)
+			(do_not_autoplace no)
+			(effects
+				(font
+					(size 1.27 1.27)
+				)
+			)
+		)
+		(property "MPN" ""
+			(at 85.09 186.69 0)
+			(hide yes)
+			(show_name no)
+			(do_not_autoplace no)
+			(effects
+				(font
+					(size 1.27 1.27)
+				)
+			)
+		)
 		(instances
 			(project "io-module"
@@
 			)
 		)
-		(property "Footprint" "CRGM Logos:Roxy 4mm"
+		(property "Footprint" "CRGM Logos:Roxy 3.5mm"
 			(at 73.66 194.818 0)
 			(hide yes)
